File: hardware/RO Flow Counter.kicad_pcb (KiCad board)
At the start: 2 copper layers, 100 x 55 mm, 74 parts, among them J1 LCD Power, J2 Conn_01x12, J3 Barrel_Jack, J5 Flow Meter, J6 Level Sensor (optional), J7 Conn_01x02, J8 Programming, K1 G5Q-1A, Q1 2N7002E, Q2 2N7002E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

Commit message: add fabrication outputs
Parts:
- added D6: WiFi, LED_SMD:LED_0805_2012Metric, F.Cu at (213.6, 62.0)
- added Q5: 2N7002E, Package_TO_SOT_SMD:SOT-23, F.Cu at (209.8, 61.2)
- added R25: 154, Resistor_SMD:R_0402_1005Metric, F.Cu at (210.6, 63.6)
- added R26: 1k, Resistor_SMD:R_0402_1005Metric, F.Cu at (205.7, 61.5)
- added R27: 10k, Resistor_SMD:R_0402_1005Metric, F.Cu at (207.3, 62.0)
- moved Q1 9.74 mm to (209.8, 71.3)
- moved R4 6.69 mm to (210.5, 73.8), turned to 180 degrees
- moved R3 5.75 mm to (210.5, 68.7), turned to 180 degrees
- moved R24 3.55 mm to (207.3, 66.9), turned to 90 degrees
- moved Q2 2.62 mm to (209.8, 66.2), turned to 270 degrees
- moved R23 2.05 mm to (207.3, 72.0)
- moved R1 1.91 mm to (205.7, 71.6)
- moved D1 0.36 mm to (213.6, 67.1), turned to 0 degrees
- moved D2 0.36 mm to (213.6, 71.9), turned to 0 degrees
- moved R2 0.19 mm to (205.7, 66.4)
Connections:
- U2 pad 16: (no net) -> /mcu/LED_WIFI
Routing:
- net /mcu/LED_WIFI: track 0.00 -> 44.7 mm, vias 0 -> 1
- net Net-(Q1-Pad1): track 17.7 -> 5.50 mm
- net Net-(Q5-Pad1): track 0.00 -> 5.60 mm
- net Net-(D6-Pad1): track 0.00 -> 2.85 mm
- net Net-(Q2-Pad3): track 4.15 -> 1.64 mm
- net /display/BACKLIGHT_LCD: track 42.9 -> 40.6 mm
- net /mcu/NORMAL_OPERATION_OUT: track 30.3 -> 28.2 mm
- net +3V3: track 283.0 -> 281.1 mm, vias 6 -> 5
- net Net-(Q5-Pad3): track 0.00 -> 1.59 mm
- net /mcu/ERROR_OUT: track 32.9 -> 31.7 mm
- net Net-(D1-Pad1): track 1.82 -> 2.90 mm
- net Net-(Q1-Pad3): track 2.58 -> 1.63 mm
- net Net-(D2-Pad1): track 2.24 -> 3.18 mm
- net Net-(Q2-Pad1): track 6.37 -> 5.45 mm
- net GND: vias 2 -> 3
Other:
- board text added: "WiFi"
