File: hardware/RO Flow Counter.sch (KiCad schematic (older format))
At the start: 29 parts, among them J7 Conn_01x02, J8 Programming, K1 G5Q-1A, Q1 2N7002E, Q2 2N7002E, Q3 2N7002E

Commit message: add fabrication outputs
Parts:
- added D6: WiFi, LED_SMD:LED_0805_2012Metric, symbol Device:LED
- added Q5: 2N7002E, Package_TO_SOT_SMD:SOT-23, symbol Transistor_FET:2N7002E
- added R25: 154, Resistor_SMD:R_0402_1005Metric, symbol Device:R
- added R26: 1k, Resistor_SMD:R_0402_1005Metric, symbol Device:R
- added R27: 10k, Resistor_SMD:R_0402_1005Metric, symbol Device:R
Connections:
- net +3V3: now also D6.2 (A)
- net GND: now also Q5.2 (S), R27.1
- new net: D6.1 (K), R25.1
- new net: Q5.3 (D), R25.2
- new net: Q5.1 (G), R26.2, R27.2
- new net mcu/LED_WIFI: R26.1
Changed lines of the file:
@@
 F15 "RESET_LCD" O R 6675 4075 50
 F16 "reset" I R 6675 5825 50
+F17 "LED_WIFI" O L 5150 5850 50
 $EndSheet
 Wire Wire Line
@@
 L power:+3.3V #PWR01
 U 1 1 62E1866C
-P 2575 2875
-F 0 "#PWR01" H 2575 2725 50  0001 C CNN
-F 1 "+3.3V" H 2590 3048 50  0000 C CNN
-F 2 "" H 2575 2875 50  0001 C CNN
-F 3 "" H 2575 2875 50  0001 C CNN
-	1    2575 2875
+P 2075 2875
+F 0 "#PWR01" H 2075 2725 50  0001 C CNN
+F 1 "+3.3V" H 2090 3048 50  0000 C CNN
+F 2 "" H 2075 2875 50  0001 C CNN
+F 3 "" H 2075 2875 50  0001 C CNN
+	1    2075 2875
 	1    0    0    -1
 $EndComp
@@
 $EndComp
 Wire Wire Line
-	2575 3100 2575 2875
+	2075 3100 2075 2875
 Wire Wire Line
 	3100 3100 2575 3100
@@
 Connection ~ 2575 5650
 Connection ~ 3100 5050
-Wire Wire Line
-	3100 5800 3100 6125
-Connection ~ 3100 5800
+$Comp
+L Device:LED D6
+U 1 1 63052445
+P 2075 3600
+F 0 "D6" H 2068 3817 50  0000 C CNN
+F 1 "WiFi" H 2068 3726 50  0000 C CNN
+F 2 "LED_SMD:LED_0805_2012Metric" H 2075 3600 50  0001 C CNN
+F 3 "~" H 2075 3600 50  0001 C CNN
+	1    2075 3600
+	0    -1   -1   0
+$EndComp
+$Comp
+L Device:R R25
+U 1 1 6305244B
+P 2075 4100
+F 0 "R25" H 2145 4146 50  0000 L CNN
+F 1 "154" H 2145 4055 50  0000 L CNN
+F 2 "Resistor_SMD:R_0402_1005Metric" V 2005 4100 50  0001 C CNN
+F 3 "~" H 2075 4100 50  0001 C CNN
+	1    2075 4100
+	1    0    0    -1
+$EndComp
+Wire Wire Line
+	2075 3950 2075 3750
+$Comp
+L Transistor_FET:2N7002E Q5
+U 1 1 63052452
+P 2175 5850
+F 0 "Q5" H 2379 5896 50  0000 L CNN
+F 1 "2N7002E" H 2379 5805 50  0000 L CNN
+F 2 "Package_TO_SOT_SMD:SOT-23" H 2375 5775 50  0001 L CIN
+F 3 "http://www.diodes.com/assets/Datasheets/ds30376.pdf" H 2175 5850 50  0001 L CNN
+	1    2175 5850
+	-1   0    0    -1
+$EndComp
+Wire Wire Line
+	2375 5850 2400 5850
+Wire Wire Line
+	2075 3100 2075 3450
+$Comp
+L Device:R R27
+U 1 1 6305245B
+P 2400 6100
+F 0 "R27" V 2193 6100 50  0000 C CNN
+F 1 "10k" V 2284 6100 50  0000 C CNN
+F 2 "Resistor_SMD:R_0402_1005Metric" V 2330 6100 50  0001 C CNN
+F 3 "~" H 2400 6100 50  0001 C CNN
+	1    2400 6100
+	-1   0    0    1
+$EndComp
+Wire Wire Line
+	2400 5950 2400 5850
+Connection ~ 2400 5850
+Wire Wire Line
+	2400 6250 2400 6350
+Wire Wire Line
+	2400 6350 2075 6350
+Wire Wire Line
+	2075 6050 2075 6350
+Wire Wire Line
+	2075 6350 2075 6500
+Connection ~ 2075 6350
+Wire Wire Line
+	2075 4250 2075 5650
+Wire Wire Line
+	2075 3100 2575 3100
+Connection ~ 2075 3100
 $Comp
 L power:GND #PWR02
 U 1 1 63073E68
-P 3100 6125
-F 0 "#PWR02" H 3100 5875 50  0001 C CNN
-F 1 "GND" H 3105 5952 50  0000 C CNN
-F 2 "" H 3100 6125 50  0001 C CNN
-F 3 "" H 3100 6125 50  0001 C CNN
-	1    3100 6125
-	1    0    0    -1
-$EndComp
+P 3100 6725
+F 0 "#PWR02" H 3100 6475 50  0001 C CNN
+F 1 "GND" H 3105 6552 50  0000 C CNN
+F 2 "" H 3100 6725 50  0001 C CNN
+F 3 "" H 3100 6725 50  0001 C CNN
+	1    3100 6725
+	1    0    0    -1
+$EndComp
+Wire Wire Line
+	3100 5800 3100 6500
+Connection ~ 3100 5800
+Wire Wire Line
+	2075 6500 3100 6500
+Connection ~ 3100 6500
+Wire Wire Line
+	3100 6500 3100 6725
+$Comp
+L Device:R R26
+U 1 1 6306EC2A
+P 4225 5850
+F 0 "R26" V 4018 5850 50  0000 C CNN
+F 1 "1k" V 4109 5850 50  0000 C CNN
+F 2 "Resistor_SMD:R_0402_1005Metric" V 4155 5850 50  0001 C CNN
+F 3 "~" H 4225 5850 50  0001 C CNN
+	1    4225 5850
+	0    1    1    0
+$EndComp
+Wire Wire Line
+	2400 5850 4075 5850
+Wire Wire Line
+	4375 5850 5150 5850
+$Comp
+L Graphic:SYM_Hot_Large #SYM1
+U 1 1 630F535C
+P 900 7400
+F 0 "#SYM1" H 900 7600 50  0001 C CNN
+F 1 "SYM_Hot_Large" H 900 7150 50  0001 C CNN
+F 2 "Custom Footprints:puppy_symbol" H 900 7200 50  0001 C CNN
+F 3 "~" H 930 7200 50  0001 C CNN
+	1    900  7400
+	1    0    0    -1
+$EndComp
